File: ddr-testbed.kicad_pcb (KiCad board)
At the start: 2 copper layers, 69.6 x 30 mm, 2 parts, among them J1 ddr4-sodimm-edge-connector, U1 MT53E256M16D1

Commit message: Fix outline
Other:
- outline, holes or cut-outs redrawn
- copper layers 2 -> 4
Changed lines of the file:
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@@
 (kicad_pcb (version 20171130) (host pcbnew 5.1.6+dfsg1-1~bpo10+1)
   (general
-    (thickness 1.6)
-    (drawings 26)
+    (thickness 1.2)
+    (drawings 24)
     (tracks 0)
     (zones 0)
@@
   (layers
     (0 F.Cu signal)
+    (1 In1.Cu power)
+    (2 In2.Cu power)
     (31 B.Cu signal)
     (32 B.Adhes user)
@@
     (tags "BGA 200 0.8x0.65")
     (attr smd)
-    (fp_text reference U1 (at 0 -8.25) (layer F.SilkS)
+    (fp_text reference U1 (at -4.47 -8.34) (layer F.SilkS)
       (effects (font (size 1 1) (thickness 0.15)))
     )
@@
       (effects (font (size 1 1) (thickness 0.15)))
     )
+    (fp_line (start -5.11 7.36) (end -5.11 -6.36) (layer F.SilkS) (width 0.12))
+    (fp_line (start 5.11 7.36) (end -5.11 7.36) (layer F.SilkS) (width 0.12))
+    (fp_line (start 5.11 -7.36) (end 5.11 7.36) (layer F.SilkS) (width 0.12))
+    (fp_line (start -4.11 -7.36) (end 5.11 -7.36) (layer F.SilkS) (width 0.12))
+    (fp_line (start 6 -8.25) (end -6 -8.25) (layer F.CrtYd) (width 0.05))
+    (fp_line (start 6 8.25) (end 6 -8.25) (layer F.CrtYd) (width 0.05))
+    (fp_line (start -6 8.25) (end 6 8.25) (layer F.CrtYd) (width 0.05))
+    (fp_line (start -6 -8.25) (end -6 8.25) (layer F.CrtYd) (width 0.05))
+    (fp_line (start 5 -7.25) (end 5 7.25) (layer F.Fab) (width 0.1))
+    (fp_line (start -4 -7.25) (end 5 -7.25) (layer F.Fab) (width 0.1))
+    (fp_line (start -5 -6.25) (end -4 -7.25) (layer F.Fab) (width 0.1))
+    (fp_line (start -5 7.25) (end -5 -6.25) (layer F.Fab) (width 0.1))
     (fp_line (start 5 7.25) (end -5 7.25) (layer F.Fab) (width 0.1))
-    (fp_line (start -5 7.25) (end -5 -6.25) (layer F.Fab) (width 0.1))
-    (fp_line (start -5 -6.25) (end -4 -7.25) (layer F.Fab) (width 0.1))
-    (fp_line (start -4 -7.25) (end 5 -7.25) (layer F.Fab) (width 0.1))
-    (fp_line (start 5 -7.25) (end 5 7.25) (layer F.Fab) (width 0.1))
-    (fp_line (start -6 -8.25) (end -6 8.25) (layer F.CrtYd) (width 0.05))
-    (fp_line (start -6 8.25) (end 6 8.25) (layer F.CrtYd) (width 0.05))
-    (fp_line (start 6 8.25) (end 6 -8.25) (layer F.CrtYd) (width 0.05))
-    (fp_line (start 6 -8.25) (end -6 -8.25) (layer F.CrtYd) (width 0.05))
-    (fp_line (start -4.11 -7.36) (end 5.11 -7.36) (layer F.SilkS) (width 0.12))
-    (fp_line (start 5.11 -7.36) (end 5.11 7.36) (layer F.SilkS) (width 0.12))
-    (fp_line (start 5.11 7.36) (end -5.11 7.36) (layer F.SilkS) (width 0.12))
-    (fp_line (start -5.11 7.36) (end -5.11 -6.36) (layer F.SilkS) (width 0.12))
     (pad AB12 smd circle (at 4.4 6.825) (size 0.27 0.27) (layers F.Cu F.Paste F.Mask)
       (net 261 "Net-(U1-PadAB12)"))
@@
     (pad A1 smd circle (at -4.4 -6.825) (size 0.27 0.27) (layers F.Cu F.Paste F.Mask)
       (net 344 "Net-(U1-PadA1)"))
-    (model ${KISYS3DMOD}/Package_BGA.3dshapes/BGA-200_10.0x14.5mm_Layout12x22_P0.80x0.65mm.wrl
-      (at (xyz 0 0 0))
+    (model ${ANT3DMDL}/BGA-200_10.0x14.5mm_Layout12x22_P0.80x0.65mm.step
+      (offset (xyz -5.15 -6.79 0.15))
       (scale (xyz 1 1 1))
       (rotate (xyz 0 0 0))
@@
   (gr_arc (start 168.85 70.75) (end 168.851561 70) (angle 89.88074856) (layer Edge.Cuts) (width 0.15))
   (gr_arc (start 168.85 99.25) (end 169.6 99.25) (angle 90) (layer Edge.Cuts) (width 0.15))
-  (gr_arc (start 139.05 99.75) (end 139.05 100) (angle 90) (layer Edge.Cuts) (width 0.15))
-  (gr_arc (start 137.55 99.75) (end 137.8 99.75) (angle 90) (layer Edge.Cuts) (width 0.15))
   (gr_arc (start 100.75 99.25) (end 100.75 100) (angle 90) (layer Edge.Cuts) (width 0.15))
-  (gr_line (start 169.6 78) (end 169.6 70.75) (layer Edge.Cuts) (width 0.15))
+  (gr_line (start 169.6 78) (end 169.600002 70.75) (layer Edge.Cuts) (width 0.15))
   (gr_arc (start 168.5 78.65) (end 167.85 78.65) (angle 90) (layer Edge.Cuts) (width 0.15))
   (gr_line (start 168.5 82) (end 169.6 82) (layer Edge.Cuts) (width 0.15))
@@
   (gr_line (start 101.75 81.35) (end 101.75 78.65) (layer Edge.Cuts) (width 0.15))
   (gr_line (start 100 82) (end 101.1 82) (layer Edge.Cuts) (width 0.15))
-  (gr_line (start 137.8 99.75) (end 137.8 96.5) (layer Edge.Cuts) (width 0.15))
+  (gr_line (start 137.55 100) (end 137.8 96.5) (layer Edge.Cuts) (width 0.15))
   (gr_line (start 138.8 99.75) (end 138.8 96.5) (layer Edge.Cuts) (width 0.15))
   (gr_arc (start 138.3 96.5) (end 137.8 96.5) (angle 180) (layer Edge.Cuts) (width 0.15))
-  (gr_line (start 139.05 100) (end 168.85 100) (layer Edge.Cuts) (width 0.15))
-  (gr_line (start 100.75 70) (end 168.85 70) (layer Edge.Cuts) (width 0.15))
+  (gr_line (start 138.8 99.75) (end 168.85 100) (layer Edge.Cuts) (width 0.15))
+  (gr_line (start 100.75 70) (end 168.851561 70) (layer Edge.Cuts) (width 0.15))
   (gr_line (start 100 99.25) (end 100 82) (layer Edge.Cuts) (width 0.15))
   (gr_line (start 169.6 99.25) (end 169.6 82) (layer Edge.Cuts) (width 0.15))
