File: ddr-testbed.sch (KiCad schematic (older format))
At the start: 9 parts, among them J1 ddr4-sodimm-edge-connector, U1 MT53E256M16D1

Commit message: Add double die configuration
Parts:
- added R? (x14): R_33R_0402, antmicro-footprints:0402-res, symbol antmicroResistors0402:R_33R_0402
Connections:
- net CK0_C: no longer U1.J9 (CK_C_A)
- net CK0_T: no longer U1.J8 (CK_T_A)
- net CS0_N: no longer U1.H4 (CS0_A)
- net ODT0: no longer U1.G2 (ODT_CA_A)
- net BG0: now reaches J1.113
- net BG1: now reaches J1.115
- net CA5_B: now reaches J1.120
- net CA5_B: now also U1.P11 (CA5_B), R?.2
- net CA3_B: now reaches J1.121
- net CA3_B: now also U1.R10 (CA3_B), R?.2
- net CA1_B: now reaches J1.122
- net CA1_B: now also U1.P2 (CA1_B), R?.2
- net CA2_B: now reaches J1.125
- net CA2_B: now also U1.R9 (CA2_B), R?.2
- net CA5_A: now reaches J1.126
- net CA5_A: now also U1.J11 (CA5_A), R?.2
- net CA0_B: now reaches J1.127
- net CA0_B: now also U1.R2 (CA0_B), R?.2
- net CA4_A: now reaches J1.128
- net CA4_A: now also U1.H11 (CA4_A), R?.2
- net DQ21: now reaches J1.45
- net DQ20: now reaches J1.46
- net DQ17: now reaches J1.49
- net DQ16: now reaches J1.50
- net DQS2_C: now reaches J1.53
- net DM2_N: now reaches J1.54
- net DQS2_T: now reaches J1.55
- net DQ22: now reaches J1.58
- net DQ23: now reaches J1.59
- net DQ18: now reaches J1.62
- net DQ19: now reaches J1.63
- net DQ28: now reaches J1.66
- net DQ29: now reaches J1.67
- net DQ24: now reaches J1.70
- net DQ25: now reaches J1.71
- net DQS3_C: now reaches J1.74
- net DM3_N: now reaches J1.75
- net DQS3_T: now reaches J1.76
- net DQ30: now reaches J1.79
- net DQ31: now reaches J1.80
- net DQ26: now reaches J1.83
- net DQ27: now reaches J1.84
- net CA3_A: now reaches J1.131
- net CA3_A: now also U1.H10 (CA3_A), R?.2
- net CA2_A: now reaches J1.132
- net CA2_A: now also U1.H9 (CA2_A), R?.2
- net CA1_A: now reaches J1.133
- net CA1_A: now also U1.J2 (CA1_A), R?.2
- net CA0_A: now reaches J1.144
- net CA0_A: now also U1.H2 (CA0_A), R?.2
- net BA1: now reaches J1.145
- net CA4_B: now reaches J1.146
- net CA4_B: now also U1.R11 (CA4_B), R?.2
- net BA0: now reaches J1.150
- net DQ24R: now reaches U1.AA11 (DQ8_B)
- net DQ16R: now reaches U1.AA2 (DQ0_B)
- net DQ23R: now reaches U1.AA4 (DQ7_B)
- net DQ31R: now reaches U1.AA9 (DQ15_B)
- net CKE0_B: now reaches U1.P4 (CKE0_B)
- net CKE0_B: now also R?.2
- net CK0_T_B: now reaches U1.P8 (CK_T_B)
- net CK0_C_B: now reaches U1.P9 (CK_C_B)
- net CS0_N_B: now reaches U1.R4 (CS0_B)
- net ODT0_B: now reaches U1.T2 (ODT_CA_B)
- net DQ27R: now reaches U1.U11 (DQ11_B)
- net DQ19R: now reaches U1.U2 (DQ3_B)
- net DQ20R: now reaches U1.U4 (DQ4_B)
- net DQ28R: now reaches U1.U9 (DQ12_B)
- net DQS3R_C: now reaches U1.V10 (DQS1_C_B)
- net DQ26R: now reaches U1.V11 (DQ10_B)
- net DQ18R: now reaches U1.V2 (DQ2_B)
- net DQS2R_C: now reaches U1.V3 (DQS0_C_B)
- net DQ21R: now reaches U1.V4 (DQ5_B)
- net DQ29R: now reaches U1.V9 (DQ13_B)
- net DQS3R_T: now reaches U1.W10 (DQS1_T_B)
- net DQS2R_T: now reaches U1.W3 (DQS0_T_B)
- net DM3R_N: now reaches U1.Y10 (DMI1_B)
- net DQ25R: now reaches U1.Y11 (DQ9_B)
- net DQ17R: now reaches U1.Y2 (DQ1_B)
- net DM2R_N: now reaches U1.Y3 (DMI0_B)
- net DQ22R: now reaches U1.Y4 (DQ6_B)
- net DQ30R: now reaches U1.Y9 (DQ14_B)
- net CKE0 renamed CKE0_A
- net CKE0_A: now also R?.2
- new net CK0_C_A: U1.J9 (CK_C_A)
- new net CK0_T_A: U1.J8 (CK_T_A)
- new net CS0_N_A: U1.H4 (CS0_A)
- new net ODT0_A: U1.G2 (ODT_CA_A)
- new net VTT: R?.1, R?.1, R?.1, R?.1, R?.1, R?.1, R?.1, R?.1, R?.1, R?.1, R?.1, R?.1, R?.1, R?.1
- no-connect marks 36 -> 16
Other:
- note added: "?"
- note added: "Second LPDDR4 die"
- note added: "Single LPDDR4 die"
- note added: "TODO: Replace with R_36"
- note removed: "Single LPDDR Chip"
- moved on the sheet: R?, U1A, U1B
