File: ddr-testbed.sch (KiCad schematic (older format))
At the start: 43 parts, among them J1 ddr4-sodimm-edge-connector, U1 MT53E256M16D1

Commit message: Redesign power supply and filtering WIP
Parts:
- removed C1: C_100p_0402, antmicro-footprints:0402-cap, symbol antmicroCapacitors0402:C_100p_0402
- removed R2: R_120R_0402, antmicro-footprints:0402-res, symbol antmicroResistors0402:R_120R_0402
- removed R3: R_0R_0402, antmicro-footprints:0402-res, symbol antmicroResistors0402:R_0R_0402
- added C11, C13, C15, C17, C19, C21, C23, C25, C27, C30, C32, C34, C36, C38, C40, C42, C44, C46, C48, C5, C50, C52, C53, C54, C55, C56, C57, C58, C59, C6, C60, C61, C8, C? (x21): C_1u_0402, antmicro-footprints:0402-cap, symbol antmicroCapacitors0402:C_1u_0402
- added C62, C63, C64, C65, C66, C67, C68, C69: C_100n_0402_6V3, antmicro-footprints:0402-cap, symbol antmicroCapacitors0402:C_100n_0402_6V3
Connections:
- net CA0_A: now also R13.1; no longer R19.1
- net CA0_B: now also R20.1; no longer R26.1
- net CA1_A: now also R14.1; no longer R18.1
- net CA1_B: now also R21.1; no longer R25.1
- net CA2_A: now also R15.1; no longer R17.1
- net CA2_B: now also R22.1; no longer R24.1
- net CA4_A: now also R17.1; no longer R15.1
- net CA4_B: now also R24.1; no longer R22.1
- net CA5_A: now also R18.1; no longer R14.1
- net CA5_B: now also R25.1; no longer R21.1
- net CKE0_A: now also R19.1; no longer R13.1
- net CKE0_B: now also R26.1; no longer R20.1
- net DDRVCC: no longer J1.111, J1.112, J1.117, J1.118, J1.123, J1.124, J1.129, J1.130, J1.135, J1.136, J1.141, J1.142, J1.147, J1.148, J1.153, J1.154, J1.159, J1.160, J1.163, R33.1, R34.1, U1.A4 (VDD2), U1.A9 (VDD2), U1.AA10 (VDDQ), U1.AA3 (VDDQ), U1.AA5 (VDDQ), U1.AA8 (VDDQ), U1.AB4 (VDD2), U1.AB9 (VDD2), U1.B10 (VDDQ), U1.B3 (VDDQ), U1.B5 (VDDQ), U1.B8 (VDDQ), U1.D1 (VDDQ), U1.D12 (VDDQ), U1.D5 (VDDQ), U1.D8 (VDDQ), U1.F1 (VDD1), U1.F10 (VDDQ), U1.F12 (VDD1), U1.F3 (VDDQ), U1.F5 (VDD2), U1.F8 (VDD2), U1.G4 (VDD1), U1.G9 (VDD1), U1.H1 (VDD2), U1.H12 (VDD2), U1.H5 (VDD2), U1.H8 (VDD2), U1.K1 (VDD2), U1.K10 (VDD2), U1.K12 (VDD2), U1.K3 (VDD2), U1.N1 (VDD2), U1.N10 (VDD2), U1.N12 (VDD2), U1.N3 (VDD2), U1.R1 (VDD2), U1.R12 (VDD2), U1.R5 (VDD2), U1.R8 (VDD2), U1.T4 (VDD1), U1.T9 (VDD1), U1.U1 (VDD1), U1.U10 (VDDQ), U1.U12 (VDD1), U1.U3 (VDDQ), U1.U5 (VDD2), U1.U8 (VDD2), U1.W1 (VDDQ), U1.W12 (VDDQ), U1.W5 (VDDQ), U1.W8 (VDDQ)
- net GND: now also C11.2, C13.2, C15.2, C17.2, C19.2, C21.2, C23.2, C25.2, C27.2, C30.2, C32.2, C34.2, C36.2, C38.2, C40.2, C42.2, C44.2, C46.2, C48.2, C5.2, C50.2, C52.2, C53.2, C54.2, C55.2, C56.2, C57.2, C58.2, C59.2, C6.2, C60.2, C61.2, C62.2, C63.2, C64.2, C65.2, C66.2, C67.2, C68.2, C69.2, C8.2, C?.2, C?.2, C?.2, C?.2, C?.2, C?.2, C?.2, C?.2, C?.2, C?.2, C?.2, C?.2, C?.2, C?.2, C?.2, C?.2, C?.2, C?.2, C?.2, C?.2, C?.2; no longer R1.2
- net ODT0_A renamed VDD1
- net VDD1: now also J1.135, J1.136, J1.141, J1.142, J1.147, J1.148, U1.F1 (VDD1), U1.F12 (VDD1), U1.G4 (VDD1), U1.G9 (VDD1), U1.T4 (VDD1), U1.T9 (VDD1), U1.U1 (VDD1), U1.U12 (VDD1), C46.1, C48.1, C50.1, C52.1, C53.1, C54.1, C55.1, C56.1, C57.1; no longer R28.1, U1.G2 (ODT_CA_A)
- new net VDD2: C58.1, C59.1, C60.1, C61.1, C?.1, C?.1, C?.1, C?.1, C?.1, C?.1, C?.1, C?.1, C?.1, C?.1, C?.1, C?.1, C?.1, C?.1, C?.1, C?.1, C?.1, C?.1, C?.1, C?.1, C?.1, J1.153, J1.154, J1.159, J1.160, J1.163, R28.1, U1.A4 (VDD2), U1.A9 (VDD2), U1.AB4 (VDD2), U1.AB9 (VDD2), U1.F5 (VDD2), U1.F8 (VDD2), U1.G2 (ODT_CA_A), U1.H1 (VDD2), U1.H12 (VDD2), U1.H5 (VDD2), U1.H8 (VDD2), U1.K1 (VDD2), U1.K10 (VDD2), U1.K12 (VDD2), U1.K3 (VDD2), U1.N1 (VDD2), U1.N10 (VDD2), U1.N12 (VDD2), U1.N3 (VDD2), U1.R1 (VDD2), U1.R12 (VDD2), U1.R5 (VDD2), U1.R8 (VDD2), U1.U5 (VDD2), U1.U8 (VDD2)
- new net VDDQ: C11.1, C13.1, C15.1, C17.1, C19.1, C21.1, C23.1, C25.1, C27.1, C30.1, C32.1, C34.1, C36.1, C38.1, C40.1, C42.1, C44.1, C5.1, C6.1, C62.1, C63.1, C64.1, C65.1, C66.1, C67.1, C68.1, C69.1, C8.1, J1.111, J1.112, J1.117, J1.118, J1.123, J1.124, J1.129, J1.130, R1.2, R33.1, R34.1, U1.AA10 (VDDQ), U1.AA3 (VDDQ), U1.AA5 (VDDQ), U1.AA8 (VDDQ), U1.B10 (VDDQ), U1.B3 (VDDQ), U1.B5 (VDDQ), U1.B8 (VDDQ), U1.D1 (VDDQ), U1.D12 (VDDQ), U1.D5 (VDDQ), U1.D8 (VDDQ), U1.F10 (VDDQ), U1.F3 (VDDQ), U1.U10 (VDDQ), U1.U3 (VDDQ), U1.W1 (VDDQ), U1.W12 (VDDQ), U1.W5 (VDDQ), U1.W8 (VDDQ)
Other:
- note added: "PLACE IT NEAR ADDRESS/COMAND/CONTROL/CLOCK ENTRY"
- note added: "Power filtering"
- note removed: "OR"
- moved on the sheet: C2, C3, C4, J1A, J1B, R1, R10, R11, R12, R13, R14, R15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

Commit message: Replace capacitors and place them on PCB
Parts:
- removed C11, C13, C15, C17, C19, C21, C23, C25, C27, C30, C32, C34, C36, C38, C40, C42, C44, C46, C48, C5, C50, C52, C53, C54, C55, C56, C57, C58, C59, C6, C60, C61, C8, C? (x21): C_1u_0402, antmicro-footprints:0402-cap, symbol antmicroCapacitors0402:C_1u_0402
- removed C62, C63, C64, C65, C66, C67, C68, C69: C_100n_0402_6V3, antmicro-footprints:0402-cap, symbol antmicroCapacitors0402:C_100n_0402_6V3
- added C1, C40, C41, C42, C5: C_10u_0402, antmicro-footprints:0402-cap, symbol antmicroCapacitors0402:C_10u_0402
- added C10, C11, C12, C13, C14, C15, C16, C17, C18, C19, C20, C21, C22, C23, C24, C25, C26, C27, C28, C29, C30, C31, C32, C33, C34, C35, C36, C37, C38, C39, C43, C45, C47, C49, C51, C52, C53, C54, C55, C56, C8, C9: C_100n_0201, antmicro-footprints:0201-res, symbol antmicroCapacitorsmisc:C_100n_0201
- added C44, C46, C48, C50, C6, C7: C_1u_0201, antmicro-footprints:0201-res, symbol antmicroCapacitorsmisc:C_1u_0201
- added FB1: BLM15PD121SN1D, antmicro-footprints:0402-res, symbol antmicroFerriteBeadsandChips:BLM15PD121SN1D
- added R2: R_10k_0402, antmicro-footprints:0402-res, symbol antmicroResistors0402:R_10k_0402
Connections:
- net labels added: VDD1_A
- wire segments 608 -> 592
Other:
- note removed: "PLACE IT NEAR ADDRESS/COMAND/CONTROL/CLOCK ENTRY"

Commit message: Preliminary LPDDR4 escape layout
Connections:
- net labels added: CK0_N, CK0_P, CK1_N, CK1_P, DQS0_N, DQS0_P, DQS1_N, DQS1_P, DQS2_N, DQS2_P, DQS3_N, DQS3_P
- net labels removed: DQS0_C, DQS0_T, DQS1_C, DQS1_T, DQS2_C, DQS2_T, DQS3_C, DQS3_T
- wire segments 592 -> 504

Commit message: LPDDR4 escape done, replaced DDR3 edge connector (requires connecting)
Parts:
- removed J1: ddr4-sodimm-edge-connector, antmicro-footprints:SODIMM_DDR4_EDGE, symbol antmicroMemoryConnectorsPCCardSockets:ddr4-sodimm-edge-connector
- added J? (x2): ddr3-sodimm-edge, antmicro-footprints:SODIMM_DDR3_EDGE, symbol antmicroMemoryConnectorsPCCardSockets:ddr3-sodimm-edge
Connections:
- wire segments 504 -> 268
- no-connect marks 65 -> 4
Other:
- note removed: "Bank adress"
- note removed: "Single LPDDR4 die"
- note removed: "What is taht pin?"
- moved on the sheet: C4, R37
