File: ddr-testbed.sch (KiCad schematic (older format))
At the start: 96 parts, among them U1 MT53E256M16D1

Commit message: Updated LPDDR4 connection on edge connector (supplies to be added)
Parts:
- removed C4: C_100n_0402_6V3, antmicro-footprints:0402-cap, symbol antmicroCapacitors0402:C_100n_0402_6V3
- removed R37: R_40R2_0402, antmicro-footprints:0402-res, symbol antmicroResistors0402:R_40R2_0402
- gave numbers to parts that had none: 1
Connections:
- net labels removed: ACT_N, ALERT_N, BA0, BA1, BG0, BG1, CK0_C, CK0_T, CK1_C, CK1_T, CS0_N, EVENT_N, PARITY, SA0, SA1, SCL, SDA, VDDSPD, VPP, VREFCA, VTT
- wire segments 268 -> 322
- no-connect marks 4 -> 0
Other:
- note removed: "Bank group\n"
- note removed: "Second LPDDR4 die"

Commit message: Passive components update, edge connector routing wip
Parts:
- added C4, C57, C58, C59, C60, C61, C62, C63, C64, C65: C_100n_0201, antmicro-footprints:0201-res, symbol antmicroCapacitorsmisc:C_100n_0201
- R11, R12, R27, R28, R29, R31, R4, R5: footprint antmicro-footprints:0402-res -> antmicro-footprints:0201-res; symbol antmicroResistors0402:R_0R_0402 -> antmicroResistorsmisc:R_0R_0201; MPN ERJ2GE0R00X -> CRCW02010000Z0ED; Manufacturer PANASONIC -> VISHAY
- R13, R14, R15, R16, R17, R18, R19: value R_40R2_0402 -> R_40R2_0201; footprint antmicro-footprints:0402-res -> antmicro-footprints:0201-res; symbol antmicroResistors0402:R_40R2_0402 -> antmicroResistorsmisc:R_40R2_0201; MPN MCWR04X40R2FTL -> CRCW020140R2FNED; Manufacturer MULTICOM PPRO -> VISHAY
- R20, R21, R22, R23, R24, R25, R26, R30, R32, R6, R7, R8, R9: footprint antmicro-footprints:0402-res -> antmicro-footprints:0201-res; symbol antmicroResistors0402:R_40R2_0402 -> antmicroResistorsmisc:R_40R2_0201; MPN MCWR04X40R2FTL -> CRCW020140R2FNED; Manufacturer MULTICOM PPRO -> VISHAY
- R33, R34: footprint antmicro-footprints:0402-res -> antmicro-footprints:0201-res; symbol antmicroResistors0402:R_80R6_0402 -> antmicroResistorsmisc:R_80R6_0201; MPN MC00625W0402180R6 -> RMCF0201FT80R6; Manufacturer MULTICOMP PRO -> VISHAY
Connections:
- wire segments 322 -> 428
Other:
- note added: "TBD: should both ODT have pull-up/pull-down resistors to test what's\nrequired?\n(NANO Pi has ODT_A pulled-up, and ODT_B NC with not populated\npull-down resistor)"

Commit message: Routing of all high speed DDR signals done
Connections:
- net labels removed: CKE_0_A, CKE_0_B
Changed lines of the file:
@@
 	5975 4700 5175 4700
 Text Label 5175 4700 0    50   ~ 0
-CKE_0_B
+CKE0_B
 Wire Wire Line
 	5975 4400 5175 4400
 Text Label 5175 4400 0    50   ~ 0
-CKE_0_A
+CKE0_A
 Text Label 5150 1625 0    50   ~ 0
 ODT0_A
@@
 CA2_B
 Text Label 15100 1875 0    50   ~ 0
-CKE0_B
+CKE_1
 Text Label 15350 1975 2    50   ~ 0
 CS_1_N

Commit message: Connect power supply to SO-DIMM connector
Connections:
- wire segments 428 -> 558
- no-connect marks 0 -> 8
