File: lpddr4-testbed.kicad_pcb (KiCad board)
At the start: 6 copper layers, 69.6 x 30 mm, 68 parts, among them IC1 PCA96408APW, IC2 AT24CS01, J1 ddr4-sodimm-edge-connector, U1 MT53E1G32D2NP-046, U2 TPS613221ADBVT

Commit message: Bumped rev on PCB
Other:
- board text added: "LPDDR4 Testbed Rev. 1.1.0 05/2021"
- board text removed: "LPDDR4 Testbed Rev. 1.0.0 01/2021"
Changed lines of the file:
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@@
-(kicad_pcb (version 20171130) (host pcbnew 5.1.9+dfsg1-1~bpo10+1)
+(kicad_pcb (version 20171130) (host pcbnew 5.1.10-88a1d61d58~88~ubuntu20.04.1)
   (general
     (thickness 1.2)
@@
   (layers
     (0 F.Cu signal)
-    (1 In1.Cu power hide)
+    (1 In1.Cu power)
     (2 In2.Cu power)
-    (3 In3.Cu signal hide)
-    (4 In4.Cu signal hide)
+    (3 In3.Cu signal)
+    (4 In4.Cu signal)
     (31 B.Cu signal)
     (32 B.Adhes user hide)
@@
   )
   (setup
-    (last_trace_width 0.2)
+    (last_trace_width 0.1)
     (user_trace_width 0.1)
     (user_trace_width 0.2)
@@
       (net 36 GND))
   )
-  (gr_text "LPDDR4 Testbed\nRev. 1.0.0  01/2021" (at 108.525 78.2) (layer F.Mask)
+  (gr_text "LPDDR4 Testbed\nRev. 1.1.0  05/2021" (at 108.525 78.2) (layer F.Mask)
     (effects (font (size 0.85 0.85) (thickness 0.18)) (justify left))
   )
-  (gr_text "LPDDR4 Testbed\nRev. 1.0.0  01/2021" (at 108.525 78.2) (layer F.Cu)
+  (gr_text "LPDDR4 Testbed\nRev. 1.1.0  05/2021" (at 108.525 78.2) (layer F.Cu)
     (effects (font (size 0.85 0.85) (thickness 0.18)) (justify left))
   )
