File: lpddr4.kicad_sch (KiCad schematic)
At the start: 43 parts, among them U1 MT53E1G32D2NP-046

Commit message: [#56947] Loclib
Parts:
- C1, C10, C11, C12, C13, C14, C15, C16, C17, C18, C19, C2, C20, C21, C22, C23, C24, C25, C26, C27, C28, C29, C3, C30, C31, C32, C33, C35, C36, C4, C5, C6, C7, C8, C9: footprint antmicro-footprints:C_0201 -> lpddr4-testbed-footprints:C_0201; symbol antmicroCapacitorsmisc:C_100n_0201 -> lpddr4-testbed:C_100n_0201
- R1, R3, R4, R5: footprint antmicro-footprints:R_0402_1005Metric -> lpddr4-testbed-footprints:R_0402_1005Metric; symbol antmicroResistors0402:R_10k_0402 -> lpddr4-testbed:R_10k_0402
- R2, R7: footprint antmicro-footprints:R_0402_1005Metric -> lpddr4-testbed-footprints:R_0402_1005Metric; symbol antmicroResistors0402:R_0R_0402 -> lpddr4-testbed:R_0R_0402
- R6: footprint antmicro-footprints:R_0402_1005Metric -> lpddr4-testbed-footprints:R_0402_1005Metric; symbol antmicroResistors0402:R_240R_0402 -> lpddr4-testbed:R_240R_0402
- U1: footprint antmicro-footprints:BGA-200_10.0x14.5mm_Layout12x22_P0.80x0.65mm -> lpddr4-testbed-footprints:BGA-200_10.0x14.5mm_Layout12x22_P0.80x0.65mm; symbol antmicroMemory:MT53E1G32D2NP-046 -> lpddr4-testbed:MT53E1G32D2NP-046
